Commit message: raise arm model pose by 1.3 meters

File: sr_description/sr_description.urdf (robot description, URDF)
Before this commit: robot arm_and_hand, 31 links, 30 joints
Joints:
- joint arm_base_joint: origin xyz=0 0 0 rpy=1.5707 0 -1.5707 -> xyz=0 0 1.3 rpy=1.5707 0 -1.5707

Commit message: expand wrist and palm collision geometry

File: sr_description/sr_description.urdf (robot description, URDF)
Before this commit: robot arm_and_hand, 31 links, 30 joints
Links:
- link palm: geometry collision box size=0.08 0.02 0.10; visual mesh filename=package://sr_description/hand/model/palm.dae scale=0.001 0.001 0.001
- link wrist: geometry collision cylinder length=0.03 radius=0.015; visual mesh filename=package://sr_description/hand/model/wrist.dae scale=0.001 0.001 0.001

Commit message: update rest of the hand collisions

File: sr_description/sr_description.urdf (robot description, URDF)
Before this commit: robot arm_and_hand, 31 links, 30 joints
Links:
- link ffknuckle: geometry collision cylinder length=0.01 radius=0.01; visual mesh filename=package://sr_description/hand/model/knuckle.dae scale=0.001 0.001 0.001
- link ffmiddle: geometry collision cylinder length=0.028 radius=0.008; visual mesh filename=package://sr_description/hand/model/F2.dae scale=0.001 0.001 0.001
- link ffproximal: geometry collision cylinder length=0.04 radius=0.01; visual mesh filename=package://sr_description/hand/model/F3.dae scale=0.001 0.001 0.001
- link lfknuckle: geometry collision cylinder length=0.01 radius=0.01; visual mesh filename=package://sr_description/hand/model/knuckle.dae scale=0.001 0.001 0.001
- link lfmetacarpal: geometry collision box size=0.019 0.019 0.05; visual mesh filename=package://sr_description/hand/model/lfmetacarpal.dae scale=0.001 0.001 0.001
- link lfmiddle: geometry collision cylinder length=0.028 radius=0.008; visual mesh filename=package://sr_description/hand/model/F2.dae scale=0.001 0.001 0.001
- link lfproximal: geometry collision cylinder length=0.04 radius=0.01; visual mesh filename=package://sr_description/hand/model/F3.dae scale=0.001 0.001 0.001
- link mfknuckle: geometry collision cylinder length=0.01 radius=0.01; visual mesh filename=package://sr_description/hand/model/knuckle.dae scale=0.001 0.001 0.001
- link mfmiddle: geometry collision cylinder length=0.028 radius=0.008; visual mesh filename=package://sr_description/hand/model/F2.dae scale=0.001 0.001 0.001
- link mfproximal: geometry collision cylinder length=0.04 radius=0.01; visual mesh filename=package://sr_description/hand/model/F3.dae scale=0.001 0.001 0.001
- link rfknuckle: geometry collision cylinder length=0.01 radius=0.01; visual mesh filename=package://sr_description/hand/model/knuckle.dae scale=0.001 0.001 0.001
- link rfmiddle: geometry collision cylinder length=0.028 radius=0.008; visual mesh filename=package://sr_description/hand/model/F2.dae scale=0.001 0.001 0.001
- link rfproximal: geometry collision cylinder length=0.04 radius=0.01; visual mesh filename=package://sr_description/hand/model/F3.dae scale=0.001 0.001 0.001
- link thbase: geometry collision sphere radius=0.0125; visual box size=0.001 0.001 0.001
- link thhub: geometry collision sphere radius=0.01; visual box size=0.001 0.001 0.001
- link thmiddle: geometry collision cylinder length=0.030 radius=0.010; collision sphere radius=0.01
- link thproximal: geometry collision cylinder length=0.04 radius=0.01; visual mesh filename=package://sr_description/hand/model/TH3_z.dae scale=0.001 0.001 0.001
